File: KiCAD/8-Bit CPU 32k.sch (KiCad schematic (older format))
At the start: 34 parts, among them J1 UART, SW1 RESET, U1 74HC04, X1 ACO-1.8432MHz

Commit message: Revision 1.3.1
Connections:
- net CLOCK renamed 1.8432MHz
Other:
- note added: "As an option, down-scaling of the\nCPU clock speed is possible here.\n"
- note added: "Ideas:\n- Make the full 128KB of the FLASH available via address jumpers.\n- Make the clock speed adjustable by down-scaling the clock with\n cascaded counters (20 bits are needed to reach 1Hz)."
- note added: "The bus is tied to $ff\nif not driven actively."
- note added: "The maximum speed is limited by\nthe access time of the control\nFLASH (70ns) or EEPROM (150ns).\n3.6864MHz (2x135ns clock cycle)\nmight be possible with FLASH,\nbut not with EEPROMs."
- moved on the sheet: C1, C10, C11, C12, C13, C14, C15, C16, C17, C18, C19, C2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
