File: KiCAD/8-Bit CPU 32k.sch (KiCad schematic (older format))
At the start: 34 parts, among them J1 UART, SW1 RESET, U1 74HC04, X1 ACO-1.8432MHz

Commit message: Revision 1.3.2
Other:
- note removed: "The maximum stable clock speed\nis limited by the access time of\nthe control FLASH (70ns), RC time\nconstant of the passive bus (70ns)\nand a small switching delay of the\nlogic gates (10ns). The system runs\nreliably up to 3MHz and becomes\nunstable at 4MHz.\nLowering the bus resistors down\nto 330Ohm MIGHT make the system\nwork at 3.6864MHz but it is NOT\nrecommended.\n"
Changed lines of the file:
@@
 Text Notes 3000 8300 0    50   ~ 0
 The bus is tied to $ff\nif not driven actively.
-Text Notes 5700 2600 0    50   ~ 0
-The maximum stable clock speed\nis limited by the access time of\nthe control FLASH (70ns), RC time\nconstant of the passive bus (70ns)\nand a small switching delay of the\nlogic gates (10ns). The system runs\nreliably up to 3MHz and becomes\nunstable at 4MHz.\nLowering the bus resistors down\nto 330Ohm MIGHT make the system\nwork at 3.6864MHz but it is NOT\nrecommended.\n
 $EndSCHEMATC
