File: KiCAD/IR.sch (KiCad schematic (older format))
At the start: 12 parts, among them U1 74HC04, U11 74HC161, U40 74HC08, U5 74HC173, U6 74HC173, U7 SST39SF010A MSB, U8 74HC173, U9 SST39SF010A LSB

Commit message: Revision 1.3.2
Parts:
- C22, C23: value 200pF -> 0pF
Changed lines of the file:
@@
 P 9200 3600
 F 0 "C23" V 9150 3500 50  0000 C CNN
-F 1 "200pF" V 9100 3750 50  0000 C CNN
+F 1 "0pF" V 9100 3750 50  0000 C CNN
 F 2 "Capacitor_THT:C_Disc_D5.0mm_W2.5mm_P2.50mm" H 9200 3600 50  0001 C CNN
 F 3 "~" H 9200 3600 50  0001 C CNN
@@
 P 6150 4150
 F 0 "C22" V 6100 4050 50  0000 C CNN
-F 1 "200pF" V 6050 4300 50  0000 C CNN
+F 1 "0pF" V 6050 4300 50  0000 C CNN
 F 2 "Capacitor_THT:C_Disc_D5.0mm_W2.5mm_P2.50mm" H 6150 4150 50  0001 C CNN
 F 3 "~" H 6150 4150 50  0001 C CNN
