File: KiCAD/RAM.sch (KiCad schematic (older format))
At the start: 8 parts, among them U1 74HC04, U26 74HC161, U28 74HC161, U30 74HC161, U31 SST39SF010A ROM, U32 CY62256 32k RAM, U33 74HC161, U44 74HC00

Commit message: Revision 1.3.1
Other:
- note added: "A separate reset of the MAR is not needed.\nDuring the time RESET is pressed,\nthe clock runs with SC=0 and PC=0.\nThis ensures that with CO|MI MAL=0."
- note added: "Writing only during\nsecond clockphase."
Changed lines of the file:
@@
 Sheet 8 9
 Title "RAM, ROM and MAR"
-Date "2021-01-18"
-Rev "1.3"
+Date "2021-02-13"
+Rev "1.3.1"
 Comp ""
 Comment1 ""
@@
 Wire Wire Line
 	1150 800  1250 800
+Text Notes 9050 1250 0    50   ~ 0
+A separate reset of the MAR is not needed.\nDuring the time RESET is pressed,\nthe clock runs with SC=0 and PC=0.\nThis ensures that with CO|MI MAL=0.
+Text Notes 4650 4650 0    50   ~ 0
+Writing only during\nsecond clockphase.
 $EndSCHEMATC
