File: KiCAD/UART_RX.sch (KiCad schematic (older format))
At the start: 8 parts, among them U1 74HC04, U19 74HC08, U20 74HC173, U34 74HC161, U35 74HC00, U37 74HC193, U39 74HC164, U41 74HC245

Commit message: Revision 1.3.1
Connections:
- net labels added: 1.8432MHz
Other:
- note added: "A falling edge in RX\nactivates the counter\nfor the duration of one\nmessage.\nThen, this shift register\nremains frozes and DR\nis signaled."
- note added: "Active only during\nsecond clockphase:\n\nOnly after reading a\nvalue, the circuit is\nreset and ready to\nreceive another char."
- note added: "If no data is present,\nreading will yield $ff\nsince 74HC245 remains\ninactive and the bus\nlines are tied HIGH."
- note added: "Sampling happens at\nthe start of a clock cycle."
- note added: "Sync. DR is needed to prevent\nDR going high during the second\nphase of the clock (this would\nallow for erasing the value without\nstoring it in a register)."
- moved on the sheet: U19C, U1C, U1E, U35A, U35B, U35C, U35D, U35E, U39, U41
