File: KiCAD/UART_RX.sch (KiCad schematic (older format))
At the start: 8 parts, among them U1 74HC04, U19 74HC08, U20 74HC173, U34 74HC161, U35 74HC00, U37 74HC193, U39 74HC164, U41 74HC245

Commit message: Revision 1.3.2
Other:
- note removed: "A falling edge in RX\nactivates the counter\nfor the duration of one\nmessage.\nThen, this shift register\nremains frozes and DR\nis signaled."
- note removed: "Active only during\nsecond clockphase:\n\nOnly after reading a\nvalue, the circuit is\nreset and ready to\nreceive another char."
- note removed: "If no data is present,\nreading will yield $ff\nsince 74HC245 remains\ninactive and the bus\nlines are tied HIGH."
- note removed: "Sampling happens at\nthe start of a clock cycle."
- note removed: "Sync. DR is needed to prevent\nDR going high during the second\nphase of the clock (this would\nallow for erasing the value without\nstoring it in a register)."
Changed lines of the file:
@@
 encoding utf-8
 Sheet 4 9
-Title ""
+Title "UART Receiver"
 Date "2021-03-10"
 Rev "1.3.2"
@@
 Wire Wire Line
 	3800 1250 3900 1250
-Text Notes 6750 4100 0    50   ~ 0
-Sync. DR is needed to prevent\nDR going high during the second\nphase of the clock (this would\nallow for erasing the value without\nstoring it in a register).
-Text Notes 6750 5800 0    50   ~ 0
-Active only during\nsecond clockphase:\n\nOnly after reading a\nvalue, the circuit is\nreset and ready to\nreceive another char.
-Text Notes 4300 5750 0    50   ~ 0
-Sampling happens at\nthe start of a clock cycle.
-Text Notes 8650 6150 0    50   ~ 0
-If no data is present,\nreading will yield $ff\nsince 74HC245 remains\ninactive and the bus\nlines are tied HIGH.
-Text Notes 750  1400 0    50   ~ 0
-A falling edge in RX\nactivates the counter\nfor the duration of one\nmessage.\nThen, this shift register\nremains frozes and DR\nis signaled.
 $EndSCHEMATC
