File: KiCAD/8-Bit CPU 32k.kicad_pcb (KiCad board)
At the start: 2 copper layers, 177.2 x 114.3 mm, 81 parts, among them J1 UART, SW1 RESET, U1 74HC04, U10 74HC173, U11 74HC161, U12 74HC86, U13 74HC283, U14 74HC283, U15 74HC245, U16 74HC86, U17 74HC173, U18 74HC02, U19 74HC08, U2 74HC173, U20 74HC173, U23 74HC245, U26 74HC161, U28 74HC161, U3 74HC173, U30 74HC161, U31 SST39SF010A ROM, U32 CY62256 32k RAM, U33 74HC161, U34 74HC161, U35 74HC00, U37 74HC193, U39 74HC164, U4 74HC245, U40 74HC08, U41 74HC245, U42 74HC161, U43 74HC165, U44 74HC00, U45 74HC165, U46 74HC161, U48 74HC00, U49 74HC161, U5 74HC173, U50 74HC245, U51 74HC161, U52 74HC161, U53 74HC245, U6 74HC173, U7 SST39SF010A MSB, U8 74HC173, U9 SST39SF010A LSB, X1 ACO-1.8432MHz

Commit message: Revision 1.3.1
Parts:
- R8, R9: value 470R -> 470
Connections:
- net CLOCK renamed 1.8432MHz

Commit message: Revision 1.3.2
Parts:
- C22, C23: value 200pF -> 0pF
Other:
- board text added: "Revision 1.3 by Carsten Herting (slu4) 2021"
- board text added: "UART configuration: 115200bps, 8 data bits, no parity bit, 1 stop bit, transmit delay 35ms/line new line: LF"
- board text removed: "Designed by Carsten Herting (slu4) 2021"
- board text removed: "UART configuration: 115200bps, 8 data bits, no parity bit, 1 stop bit, no flow control, transmit delay 20ms per line new line: LF, local echo off"
Changed lines of the file:
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@@
       (drillshape 0)
       (scaleselection 1)
-      (outputdirectory "Gerbers/"))
+      (outputdirectory "Minimal_1.3_Gerbers/"))
   )
   (net 0 "")
@@
       (effects (font (size 1 1) (thickness 0.15)))
     )
-    (fp_text value 200pF (at 1.27 -2.54) (layer F.SilkS)
+    (fp_text value 0pF (at 1.27 -2.54) (layer F.SilkS)
       (effects (font (size 1 1) (thickness 0.15)))
     )
@@
       (effects (font (size 1 1) (thickness 0.15)))
     )
-    (fp_text value 200pF (at 1.25 2.5) (layer F.SilkS)
+    (fp_text value 0pF (at 1.25 2.5) (layer F.SilkS)
       (effects (font (size 1 1) (thickness 0.15)))
     )
@@
     (effects (font (size 0.75 0.75) (thickness 0.125)))
   )
-  (gr_text "UART configuration:\n115200bps, 8 data bits,\nno parity bit, 1 stop bit,\nno flow control,\ntransmit delay 20ms per line\nnew line: LF, local echo off" (at 199.136 127.508) (layer F.SilkS)
+  (gr_text "UART configuration:\n115200bps, 8 data bits,\nno parity bit, 1 stop bit,\ntransmit delay 35ms/line\nnew line: LF" (at 200.025 127.508) (layer F.SilkS)
     (effects (font (size 0.75 0.75) (thickness 0.125)) (justify left))
   )
@@
     (effects (font (size 1 1) (thickness 0.15)))
   )
-  (gr_text "Designed by Carsten Herting (slu4) 2021" (at 172.72 127.635) (layer F.SilkS)
+  (gr_text "Revision 1.3 by Carsten Herting (slu4) 2021" (at 173.355 127.635) (layer F.SilkS)
     (effects (font (size 1 1) (thickness 0.125)))
   )
